Commit message: URDF package with joint state pub gui

File: flightsim_ws/src/abb_irb7600/description/urdf/common_materials.xacro (robot description, xacro)
@@ -1,5 +1,5 @@
 <?xml version="1.0"?>
 <robot xmlns:xacro="http://ros.org/wiki/xacro">
-  <xacro:include filename="$(find abb_resources)/urdf/common_colours.xacro"/>
+  <xacro:include filename="$(find abb_irb7600)/description/urdf/common_colours.xacro"/>
   <xacro:macro name="material_abb_orange">
     <material name="">

File: flightsim_ws/src/abb_irb7600/description/urdf/irb7600_150_350_macro.xacro (robot description, xacro)
@@ -1,5 +1,5 @@
 <?xml version="1.0"?>
 <robot xmlns:xacro="http://ros.org/wiki/xacro">
-  <xacro:include filename="$(find abb_resources)/urdf/common_materials.xacro"/>
+  <xacro:include filename="$(find abb_irb7600)/description/urdf/common_materials.xacro"/>
   <xacro:macro name="abb_irb7600_150_350" params="prefix">
     <!-- link list -->
@@ -136,4 +136,42 @@
         </geometry>
         <xacro:material_abb_yellow />
+      </collision>
+    </link>
+    <link name="${prefix}pilot_cabin_link">
+      <visual>
+        <origin xyz="0 0 0" rpy="0 0 0"/>
+        <geometry>
+          <box size="1 1 1.4"/>
+        </geometry>
+        <xacro:material_abb_pebble_gray />
+      </visual>
+      <collision>
+        <origin xyz="0 0 0" rpy="0 0 0"/>
+        <geometry>
+          <box size="1 1 1.4"/>
+        </geometry>
+      </collision>
+      <inertial>
+        <origin xyz="0 0 0" rpy="0 0 0"/>
+        <mass value="150.0"/>  <!-- mass in kilograms -->
+        <inertia
+          ixx="39.67" ixy="0.0" ixz="0.0"
+          iyy="39.67" iyz="0.0"
+          izz="25.0"/>
+      </inertial>
+    </link>
+    <link name="${prefix}wings_link">
+      <visual>
+        <origin xyz="0 0 0" rpy="0 0 0"/>
+        <geometry>
+          <box size="0.1 2 0.2"/>
+        </geometry>
+        <xacro:material_abb_yellow/>
+      </visual>
+      <collision>
+        <origin xyz="0 0 0" rpy="0 0 0"/>
+        <geometry>
+          <box size="0.1 2 0.2"/>
+        </geometry>
       </collision>
     </link>
@@ -209,4 +247,15 @@
       <child link="${prefix}tool0" />
     </joint>
+    <!--endeffektor pilot cabin joint-->
+    <joint name="${prefix}joint_pilot_cabin" type="fixed">
+      <origin xyz="0 0 0.7" rpy="0 0 0"/>
+      <parent link="${prefix}tool0"/>
+      <child link="${prefix}pilot_cabin_link"/>
+    </joint>
+    <joint name="${prefix}joint_wings" type="fixed">
+      <origin xyz="0 0 0.2" rpy="0 0 0"/>
+      <parent link="${prefix}tool0"/>
+      <child link="${prefix}wings_link"/>
+    </joint>
   </xacro:macro>
 </robot>
