Commit message: added gazebo functionality, still look to slim down the files

File: flightsim_ws/src/abb_irb7600/description/urdf/irb7600_150_350.urdf.xacro (robot description, xacro)
@@ -2,4 +2,5 @@
 <robot name="abb_irb7600_150_350" xmlns:xacro="http://ros.org/wiki/xacro">
   <xacro:include filename="$(find abb_irb7600)/description/urdf/irb7600_150_350_macro.xacro"/>
+  <xacro:include filename="$(find abb_irb7600)/description/urdf/irb7600_150_350.gazebo"/>
   <xacro:abb_irb7600_150_350 prefix=""/>
 </robot>

File: flightsim_ws/src/abb_irb7600/description/urdf/irb7600_150_350_macro.xacro (robot description, xacro)
@@ -4,18 +4,26 @@
   <xacro:macro name="abb_irb7600_150_350" params="prefix">
     <!-- link list -->
+    <link name="world"/>
     <link name="${prefix}base_link">
       <visual>
         <origin xyz="0 0 0" rpy="0 0 0"/>
         <geometry>
-          <mesh filename="package://abb_irb7600/description/meshes/irb7600/visual/base_link.stl"/>
-        </geometry>
-        <xacro:material_abb_orange />
-      </visual>
-      <collision>
-        <geometry>
-          <mesh filename="package://abb_irb7600/description/meshes/irb7600/collision/base_link.stl"/>
-        </geometry>
-        <xacro:material_abb_orange />
-      </collision>
+          <mesh filename="$(find abb_irb7600)/description/meshes/base_link.stl"/>
+        </geometry>
+        <xacro:material_abb_orange />
+      </visual>
+      <collision>
+        <geometry>
+          <mesh filename="$(find abb_irb7600)/description/meshes/base_link.stl"/>
+        </geometry>
+      </collision>
+      <inertial>
+        <mass value="1000.0"/>
+        <origin xyz="0 0 0" rpy="0 0 0"/>
+        <inertia
+          ixx="0.01" ixy="0.0" ixz="0.0"
+          iyy="0.01" iyz="0.0"
+          izz="0.01"/>
+      </inertial>
     </link>
     <link name="${prefix}link_1">
@@ -23,15 +31,22 @@
         <origin xyz="0 0 0" rpy="0 0 0"/>
         <geometry>
-          <mesh filename="package://abb_irb7600/description/meshes/irb7600/visual/link_1.stl"/>
-        </geometry>
-        <xacro:material_abb_orange />
-      </visual>
-      <collision>
-        <origin xyz="0 0 0" rpy="0 0 0"/>
-        <geometry>
-          <mesh filename="package://abb_irb7600/description/meshes/irb7600/collision/link_1.stl"/>
-        </geometry>
-        <xacro:material_abb_yellow />
-      </collision>
+          <mesh filename="$(find abb_irb7600)/description//meshes/link_1.stl"/>
+        </geometry>
+        <xacro:material_abb_orange />
+      </visual>
+      <collision>
+        <origin xyz="0 0 0" rpy="0 0 0"/>
+        <geometry>
+          <mesh filename="$(find abb_irb7600)/description/meshes/link_1.stl"/>
+        </geometry>
+      </collision>
+      <inertial>
+        <mass value="500.0"/>
+        <origin xyz="0 0 0" rpy="0 0 0"/>
+        <inertia
+          ixx="0.01" ixy="0.0" ixz="0.0"
+          iyy="0.01" iyz="0.0"
+          izz="0.01"/>
+      </inertial>
     </link>
     <link name="${prefix}link_2">
@@ -39,15 +54,22 @@
         <origin xyz="0 0 0" rpy="0 0 0"/>
         <geometry>
-          <mesh filename="package://abb_irb7600/description/meshes/irb7600/visual/link_2.stl"/>
-        </geometry>
-        <xacro:material_abb_orange />
-      </visual>
-      <collision>
-        <origin xyz="0 0 0" rpy="0 0 0"/>
-        <geometry>
-          <mesh filename="package://abb_irb7600/description/meshes/irb7600/collision/link_2.stl"/>
-        </geometry>
-        <xacro:material_abb_yellow />
-      </collision>
+          <mesh filename="$(find abb_irb7600)/description/meshes/link_2.stl"/>
+        </geometry>
+        <xacro:material_abb_orange />
+      </visual>
+      <collision>
+        <origin xyz="0 0 0" rpy="0 0 0"/>
+        <geometry>
+          <mesh filename="$(find abb_irb7600)/description/meshes/link_2.stl"/>
+        </geometry>
+      </collision>
+      <inertial>
+        <mass value="200.0"/>
+        <origin xyz="0 0 0" rpy="0 0 0"/>
+        <inertia
+          ixx="0.01" ixy="0.0" ixz="0.0"
+          iyy="0.01" iyz="0.0"
+          izz="0.01"/>
+      </inertial>
     </link>
     <link name="${prefix}link_3">
@@ -55,15 +77,22 @@
         <origin xyz="0 0 0" rpy="0 0 0"/>
         <geometry>
-          <mesh filename="package://abb_irb7600/description/meshes/irb7600/visual/link_3.stl"/>
-        </geometry>
-        <xacro:material_abb_orange />
-      </visual>
-      <collision>
-        <origin xyz="0 0 0" rpy="0 0 0"/>
-        <geometry>
-          <mesh filename="package://abb_irb7600/description/meshes/irb7600/collision/link_3.stl"/>
-        </geometry>
-        <xacro:material_abb_yellow />
-      </collision>
+          <mesh filename="$(find abb_irb7600)/description/meshes/link_3.stl"/>
+        </geometry>
+        <xacro:material_abb_orange />
+      </visual>
+      <collision>
+        <origin xyz="0 0 0" rpy="0 0 0"/>
+        <geometry>
+          <mesh filename="$(find abb_irb7600)/description/meshes/link_3.stl"/>
+        </geometry>
+      </collision>
+      <inertial>
+        <mass value="100.0"/>
+        <origin xyz="0 0 0" rpy="0 0 0"/>
+        <inertia
+          ixx="0.01" ixy="0.0" ixz="0.0"
+          iyy="0.01" iyz="0.0"
+          izz="0.01"/>
+      </inertial>
     </link>
     <link name="${prefix}link_4">
@@ -71,5 +100,5 @@
         <origin xyz="2.012 0 0" rpy="0 0 0"/>
         <geometry>
-          <mesh filename="package://abb_irb7600/description/meshes/irb7600_150_350/visual/link_4.stl"/>
+          <mesh filename="$(find abb_irb7600)/description/meshes/link_4.stl"/>
         </geometry>
         <xacro:material_abb_orange />
@@ -78,5 +107,5 @@
         <origin xyz="2.012 0 0" rpy="0 0 0"/>
         <geometry>
-          <mesh filename="package://abb_irb7600/description/meshes/irb7600_150_350/visual/abb_logos.stl"/>
+          <mesh filename="$(find abb_irb7600)/description/meshes/abb_logos.stl"/>
         </geometry>
         <xacro:material_abb_black />
@@ -85,8 +114,15 @@
         <origin xyz="2.012 0 0" rpy="0 0 0"/>
         <geometry>
-          <mesh filename="package://abb_irb7600/description/meshes/irb7600_150_350/collision/link_4.stl"/>
-        </geometry>
-        <xacro:material_abb_yellow />
-      </collision>
+          <mesh filename="$(find abb_irb7600)/description/meshes/link_4.stl"/>
+        </geometry>
+      </collision>
+      <inertial>
+        <mass value="50.0"/>
+        <origin xyz="0 0 0" rpy="0 0 0"/>
+        <inertia
+          ixx="0.01" ixy="0.0" ixz="0.0"
+          iyy="0.01" iyz="0.0"
+          izz="0.01"/>
+      </inertial>
     </link>
     <link name="${prefix}link_5">
@@ -94,15 +130,22 @@
         <origin xyz="0 0 0" rpy="0 0 0"/>
         <geometry>
-          <mesh filename="package://abb_irb7600/description/meshes/irb7600/visual/link_5.stl"/>
-        </geometry>
-        <xacro:material_abb_orange />
-      </visual>
-      <collision>
-        <origin xyz="0 0 0" rpy="0 0 0"/>
-        <geometry>
-          <mesh filename="package://abb_irb7600/description/meshes/irb7600/collision/link_5.stl"/>
-        </geometry>
-        <xacro:material_abb_yellow />
-      </collision>
+          <mesh filename="$(find abb_irb7600)/description/meshes/link_5.stl"/>
+        </geometry>
+        <xacro:material_abb_orange />
+      </visual>
+      <collision>
+        <origin xyz="0 0 0" rpy="0 0 0"/>
+        <geometry>
+          <mesh filename="$(find abb_irb7600)/description/meshes/link_5.stl"/>
+        </geometry>
+      </collision>
+      <inertial>
+        <mass value="25.0"/>
+        <origin xyz="0 0 0" rpy="0 0 0"/>
+        <inertia
+          ixx="0.01" ixy="0.0" ixz="0.0"
+          iyy="0.01" iyz="0.0"
+          izz="0.01"/>
+      </inertial>
     </link>
     <link name="${prefix}link_6">
@@ -110,5 +153,5 @@
         <origin xyz="0 0 0" rpy="0 0 0"/>
         <geometry>
-          <mesh filename="package://abb_irb7600/description/meshes/irb7600/visual/link_6.stl"/>
+          <mesh filename="$(find abb_irb7600)/description/meshes/link_6.stl"/>
         </geometry>
         <xacro:material_abb_black />
@@ -117,8 +160,15 @@
         <origin xyz="0 0 0" rpy="0 0 0"/>
         <geometry>
-          <mesh filename="package://abb_irb7600/description/meshes/irb7600/collision/link_6.stl"/>
-        </geometry>
-        <xacro:material_abb_black />
-      </collision>
+          <mesh filename="$(find abb_irb7600)/description/meshes/link_6.stl"/>
+        </geometry>
+      </collision>
+      <inertial>
+        <mass value="25.0"/>
+        <origin xyz="0 0 0" rpy="0 0 0"/>
+        <inertia
+          ixx="0.01" ixy="0.0" ixz="0.0"
+          iyy="0.01" iyz="0.0"
+          izz="0.01"/>
+      </inertial>
     </link>
     <link name="${prefix}balancer_piston">
@@ -126,15 +176,22 @@
         <origin xyz="0 0 0" rpy="0 0 0"/>
         <geometry>
-          <mesh filename="package://abb_irb7600/description/meshes/irb7600/visual/balancer_piston.stl"/>
-        </geometry>
-        <xacro:material_abb_orange />
-      </visual>
-      <collision>
-        <origin xyz="0 0 0" rpy="0 0 0"/>
-        <geometry>
-          <mesh filename="package://abb_irb7600/description/meshes/irb7600/collision/balancer_piston.stl"/>
-        </geometry>
-        <xacro:material_abb_yellow />
-      </collision>
+          <mesh filename="$(find abb_irb7600)/description/meshes/balancer_piston.stl"/>
+        </geometry>
+        <xacro:material_abb_orange />
+      </visual>
+      <collision>
+        <origin xyz="0 0 0" rpy="0 0 0"/>
+        <geometry>
+          <mesh filename="$(find abb_irb7600)/description/meshes/balancer_piston.stl"/>
+        </geometry>
+      </collision>
+      <inertial>
+        <mass value="25.0"/>
+        <origin xyz="0 0 0" rpy="0 0 0"/>
+        <inertia
+          ixx="0.01" ixy="0.0" ixz="0.0"
+          iyy="0.01" iyz="0.0"
+          izz="0.01"/>
+      </inertial>
     </link>
     <link name="${prefix}pilot_cabin_link">
@@ -175,7 +232,19 @@
         </geometry>
       </collision>
+      <inertial>
+        <mass value="1.0"/>
+        <origin xyz="0 0 0" rpy="0 0 0"/>
+        <inertia
+          ixx="0.01" ixy="0.0" ixz="0.0"
+          iyy="0.01" iyz="0.0"
+          izz="0.01"/>
+      </inertial>
     </link>
     <!-- end of link list -->
     <!-- joint list -->
+    <joint name="world_joint" type="fixed">
+      <parent link="world"/>
+      <child link="base_link"/>
+    </joint>
     <joint name="${prefix}joint_1" type="revolute">
       <origin xyz="0 0 0" rpy="0 0 0"/>
@@ -228,8 +297,8 @@
     <!-- ROS-Industrial 'base' frame: base_link to ABB World Coordinates transform -->
     <link name="${prefix}base" />
-    <joint name="${prefix}base_link-base" type="fixed">
-      <origin xyz="0 0 0" rpy="0 0 0"/>
-      <parent link="${prefix}base_link"/>
-      <child link="${prefix}base"/>
+    <joint name="base_link-base" type="fixed">
+      <origin rpy="0 0 0" xyz="0 0 0"/>
+      <parent link="base_link"/>
+      <child link="base"/>
     </joint>
     <!-- ROS-Industrial 'flange' frame: attachment point for EEF models -->
