Commit message: added Qt interface

File: abbflightsim_ws/src/irb7600_description/urdf/mech/irb7600_150_350_macro.xacro (robot description, xacro)
@@ -88,10 +88,10 @@
       </collision>
       <inertial>
-        <mass value="200.0"/>
-        <origin xyz="0 0 0" rpy="0 0 0"/>
-        <inertia
-          ixx="40.0" ixy="0.0" ixz="0.0"
-          iyy="40.0" iyz="0.0"
-          izz="40.0"/>
+        <mass value="50.0"/>
+        <origin xyz="0 0 0" rpy="0 0 0"/>
+        <inertia
+          ixx="10.0" ixy="0.0" ixz="0.0"
+          iyy="10.0" iyz="0.0"
+          izz="10.0"/>
       </inertial>
     </link>
